File: new/unikbd/hardware/kbd/unikbd-keys.kicad_pcb (KiCad board)
At the start: 2 copper layers, 304.8 x 101.6 mm, 122 parts, among them J1 Conn_02x20_Odd_Even, SW1 Clear, SW10 Bracket_Open, SW11 6, SW12 Y, SW13 Return, SW14 Dash, SW15 5, SW16 T, SW17 Line Feed, SW18 Colon, SW19 4, SW2 Repeat, SW20 R, SW21 O, SW22 0, SW23 3, SW24 E, SW25 L, SW26 9, SW27 2, SW28 W, SW29 Period, SW3 Tilde, SW30 8, SW31 1, SW32 Ampersand, SW33 Break, SW34 Rubout, SW35 R_Shift, SW36 P, SW37 Comma, SW38 K, SW39 L_Shift, SW4 I, SW40 Semicolon, SW41 M, SW42 J, SW43 Fwd_Slash, SW44 N, SW45 H, SW46 SPACE, SW47 B, SW48 G, SW49 ESC, SW5 Here_is, SW50 Z, SW51 V, SW52 F, SW53 CTRL, SW54 A, SW55 C, SW56 D, SW57 Backslash, SW58 Q, SW59 X, SW6 Bracket_Close, SW60 S, SW7 7, SW8 U, SW9 Shift_Lock

Commit message: update 502 files to fix missing traces
Parts:
- removed D33, D35: 1N4148, Diode_THT:D_DO-35_SOD27_P7.62mm_Horizontal
Connections:
- SW32 pad 1: /Col0 -> Net-(J1-Pad6)
- SW32 pad 2: Net-(D33-Pad2) -> Net-(J1-Pad8)
- SW34 pad 1: /Col0 -> Net-(J1-Pad10)
- SW34 pad 2: Net-(D35-Pad2) -> Net-(J1-Pad12)
Routing:
- net Net-(J1-Pad6): track 0.00 -> 65.9 mm
- net Net-(J1-Pad10): track 0.00 -> 63.8 mm
- net Net-(J1-Pad8): track 0.00 -> 61.5 mm
- net /Col0: track 177.9 -> 124.5 mm, vias 1 -> 2
- net Net-(J1-Pad12): track 0.00 -> 50.0 mm
- net Net-(D1-Pad1): track 235.5 -> 248.9 mm
- net /Col1: track 361.4 -> 373.9 mm
- net Net-(D35-Pad2): track 9.86 -> 0.00 mm
- net Net-(D33-Pad2): track 9.63 -> 0.00 mm
- net Net-(D1-Pad2): track 229.4 -> 238.3 mm
- net /Row1: track 366.7 -> 361.2 mm
- net /Row0: track 372.2 -> 367.7 mm, vias 4 -> 5
- net /Col2: track 468.5 -> 470.5 mm
- net /Col4: track 321.5 -> 319.7 mm
- net /Col5: track 463.5 -> 464.5 mm
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Other:
- outline, holes or cut-outs redrawn
